Commit message: attempting to add world frame in urdf, wrote untested code for bending motion

File: urdf/val_valkyrie_D.urdf (robot description, URDF)
Before this commit: robot ValkyrieD, 69 links, 68 joints
Links:
- added link world
Joints:
- added joint fixed: type fixed, parent world, child pelvis
